File: bitcart.kicad_pcb (KiCad board)
At the start: 4 copper layers, 136.6 x 54.6 mm, 78 parts, among them J1 Conn_01x03, J11 USB_OTG, J17 Molex 470531000, J2 Conn_02x07_Odd_Even, J3 Conn_01x03, Q1 SI7430DP, Q2 TL432DBZ, Q4 MMBTA06LT1G, T1 7491194912, U1 MP8008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

Commit message: started routing PoE
Parts:
- removed D4: LED Green, LED_SMD:LED_0603_1608Metric
- removed D5: LED Red, LED_SMD:LED_0603_1608Metric
- removed R14, R15: 2.2K 1%, Resistor_SMD:R_0402_1005Metric
- removed R16: 36K 1%, Resistor_SMD:R_0402_1005Metric
- removed R5, R6: 1k, Resistor_SMD:R_0402_1005Metric
- added D20: LED Red, LED_SMD:LED_0603_1608Metric, F.Cu at (111.4, 171.0)
- added D21: LED Green, LED_SMD:LED_0603_1608Metric, F.Cu at (116.0, 171.9)
- added R30: 2.2K 1%, Resistor_SMD:R_0402_1005Metric, F.Cu at (177.9, 149.2)
- added R31: 2.2K 1%, Resistor_SMD:R_0402_1005Metric, F.Cu at (175.0, 149.2)
- added R32: 36K 1%, Resistor_SMD:R_0402_1005Metric, F.Cu at (176.7, 152.6)
- added R33: 1k, Resistor_SMD:R_0402_1005Metric, F.Cu at (119.0, 167.5)
- added R34: 1k, Resistor_SMD:R_0402_1005Metric, F.Cu at (116.0, 167.5)
- moved R8 103.7 mm to (257.9, 218.7), turned to 180 degrees
- moved R10 89.9 mm to (251.0, 210.4), turned to -90 degrees
- moved U1 87.8 mm to (251.5, 218.0), turned to 90 degrees
- moved D3 68.2 mm to (243.5, 213.6), turned to -90 degrees
- moved C1 67.3 mm to (256.3, 200.6), turned to -90 degrees
- moved R20 65.8 mm to (258.6, 213.5), turned to -90 degrees
- moved R13 64.4 mm to (262.6, 200.6), turned to 90 degrees
- moved C11 61.2 mm to (299.4, 225.2), turned to -90 degrees
- moved D9 47.8 mm to (256.3, 213.5), turned to 90 degrees
- moved U10 47.5 mm to (207.6, 203.6), turned to -90 degrees
- moved R3 46.3 mm to (249.4, 223.0), turned to -90 degrees
- moved C6 46.0 mm to (252.5, 213.3), turned to 90 degrees
- moved R9 45.5 mm to (253.9, 205.7), turned to -90 degrees
- moved R4 37.5 mm to (245.9, 218.2), turned to -90 degrees
- moved C1-2 36.4 mm to (252.2, 200.6), turned to -90 degrees
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Connections:
- net Net-(C10-Pad1) renamed /PoE/NS
- net Net-(C2-Pad1) renamed /PoE/LS
- net Net-(R10-Pad1) renamed /PoE/ISQ
Routing:
- net /PoE/TR1_TAP: track 0.00 -> 31.6 mm, vias 0 -> 1
- net /PoE/TR2_TAP: track 0.00 -> 31.1 mm, vias 0 -> 1
- net /PoE/VDD: track 0.00 -> 30.9 mm, vias 0 -> 2
- net /PoE/COMP: track 0.00 -> 27.3 mm, vias 0 -> 2
- net /+5v: track 0.00 -> 23.4 mm, vias 0 -> 2
- net /PoE/W4: track 0.00 -> 16.3 mm
- net Net-(D9-Pad1): track 0.00 -> 15.3 mm, vias 0 -> 2
- net /PoE/VIN: track 0.00 -> 15.2 mm
- net Net-(C12-Pad1): track 0.00 -> 14.4 mm
- net Net-(C11-Pad2): track 0.00 -> 13.6 mm
- net /PoE/TR0_TAP: track 0.00 -> 13.0 mm
- net /PoE/TR3_TAP: track 0.00 -> 12.8 mm
- net /PoE/GND1: track 0.00 -> 11.0 mm
- net Net-(R21-Pad2): track 0.00 -> 10.3 mm
- net Net-(C8-Pad2): track 0.00 -> 8.22 mm
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- added copper zone on F.Cu, net /+5v
- added copper zone on F.Cu, net /PoE/GND1
- added copper zone on F.Cu, net /PoE/ISQ
- added copper zone on F.Cu, net /PoE/LS
- added copper zone on F.Cu, net /PoE/NS
- added copper zone on F.Cu, net /PoE/VDD
- added copper zone on F.Cu, net /PoE/VSS
- added copper zone on F.Cu, net /PoE/W1
- added copper zone on F.Cu, net GND
- removed copper zone on In2.Cu, net /+3.3v
- removed copper zone on In1.Cu, net GND
- removed copper zone on In2.Cu, net GND
